Commit message: Added Pisa/IIT Soft-Hand model to the mobile manipulator.

File: gazebo_oru/cititruck/cititruck_description/urdf/cititruck_manipulator.xacro (robot description, xacro)
@@ -354,4 +354,7 @@
     <origin xyz="0 0 0.0" rpy="0 0 0"/>
   </xacro:soft_hand>-->
+  <xacro:soft_hand parent="right_arm_7_link" name="right_hand" left="false" withAdaptiveTransmission="false" useMimicTag="true">
+    <origin xyz="0 0 0.0" rpy="0 0 0"/>
+  </xacro:soft_hand>
   <link name="ft_surface">
       <inertial>

Commit message: fixed hand orientation in cititruck_manipulator and initial joint configuration

File: gazebo_oru/cititruck/cititruck_description/urdf/cititruck_manipulator.xacro (robot description, xacro)
@@ -355,5 +355,5 @@
   </xacro:soft_hand>-->
   <xacro:soft_hand parent="right_arm_7_link" name="right_hand" left="false" withAdaptiveTransmission="false" useMimicTag="true">
-    <origin xyz="0 0 0.0" rpy="0 0 0"/>
+    <origin xyz="0 0 0.0" rpy="0 0 3.14159"/>
   </xacro:soft_hand>
   <link name="ft_surface">

Commit message: changed initial robot configuration accordingly to hand pose

File: gazebo_oru/cititruck/cititruck_description/urdf/cititruck_manipulator.xacro (robot description, xacro)
@@ -355,5 +355,5 @@
   </xacro:soft_hand>-->
   <xacro:soft_hand parent="right_arm_7_link" name="right_hand" left="false" withAdaptiveTransmission="false" useMimicTag="true">
-    <origin xyz="0 0 0.0" rpy="0 0 3.14159"/>
+    <origin xyz="0 0 0.0" rpy="0 0 0"/>
   </xacro:soft_hand>
   <link name="ft_surface">
