Commit message: Adding sensor calibration for big truck

File: gazebo_oru/cititruck/cititruck_description/urdf/BTruck.xacro (robot description, xacro)
@@ -5,4 +5,6 @@
   <!-- Import Rviz colors -->
   <xacro:include filename="$(find cititruck_description)/urdf/materials.xacro" />
+  <!-- Adds extra joints for calibration of sensors -->
+  <xacro:include filename="$(find cititruck_description)/urdf/sensor_calibration_assembly.xacro" />
   <xacro:property name="forks_pidP" value="2000" />
   <xacro:property name="forks_pidI" value="0" />
@@ -14,29 +16,29 @@
   <xacro:property name="M_PI" value="3.1415927" />
  <!-- BTruck dimension paraemters -->
-	<xacro:property name="x" value="0.786" />
-	<xacro:property name="y" value="1.604" />
-	<xacro:property name="m1" value="0.055" />
-	<xacro:property name="b1" value="0.79" />
-	<xacro:property name="l2" value="1.186" />
-	<xacro:property name="h3" value="1.712" />
-	<xacro:property name="b11" value="0.38" />
-	<xacro:property name="h13" value="0.091" />
-	<xacro:property name="e" value="0.18" />
-	<xacro:property name="l" value="1.2" />
-	<xacro:property name="x_pilar" value="0.24" />
-	<xacro:property name="y_pilar" value="0.05" /> <!-- to check -->
-	<xacro:property name="z_pilar" value="2.25" />
-	<xacro:property name="y_sensor_platform" value="0.64" /> <!--external distance between pilars-->
-	<xacro:property name="b5" value="0.55" />
-	<xacro:property name="x_sensor_bar" value="${x_pilar + 0.05}" />
-	<xacro:property name="y_sensor_bar" value="${y_sensor_platform - 2*y_pilar}" />
-	<xacro:property name="z_sensor_bar" value="0.04" />
-	<xacro:property name="rear_wheel_diameter" value="0.085" />
-	<xacro:property name="rear_wheel_length" value="0.075" />
-	<xacro:property name="front_wheel_length" value="0.05" />
-	<xacro:property name="front_wheel_diameter" value="0.150" />
-	<xacro:property name="x_sick" value="0.1" />
-	<xacro:property name="y_sick" value="0.1" />
-	<xacro:property name="z_sick" value="0.1" />
+    <xacro:property name="x" value="0.786" />
+    <xacro:property name="y" value="1.604" />
+    <xacro:property name="m1" value="0.055" />
+    <xacro:property name="b1" value="0.79" />
+    <xacro:property name="l2" value="1.186" />
+    <xacro:property name="h3" value="1.712" />
+    <xacro:property name="b11" value="0.38" />
+    <xacro:property name="h13" value="0.091" />
+    <xacro:property name="e" value="0.18" />
+    <xacro:property name="l" value="1.2" />
+    <xacro:property name="x_pilar" value="0.24" />
+    <xacro:property name="y_pilar" value="0.05" /> <!-- to check -->
+    <xacro:property name="z_pilar" value="2.25" />
+    <xacro:property name="y_sensor_platform" value="0.64" /> <!--external distance between pilars-->
+    <xacro:property name="b5" value="0.55" />
+    <xacro:property name="x_sensor_bar" value="${x_pilar + 0.05}" />
+    <xacro:property name="y_sensor_bar" value="${y_sensor_platform - 2*y_pilar}" />
+    <xacro:property name="z_sensor_bar" value="0.04" />
+    <xacro:property name="rear_wheel_diameter" value="0.085" />
+    <xacro:property name="rear_wheel_length" value="0.075" />
+    <xacro:property name="front_wheel_length" value="0.05" />
+    <xacro:property name="front_wheel_diameter" value="0.150" />
+    <xacro:property name="x_sick" value="0.1" />
+    <xacro:property name="y_sick" value="0.1" />
+    <xacro:property name="z_sick" value="0.1" />
   <!-- base_footprint is a fictitious link(frame) that is on the ground right below base_link origin, navigation stack dedpends on this frame and KDL needs a root link without any inteltia -->
     <link name="base_footprint">
@@ -87,5 +89,5 @@
           <box size="${l} ${e} ${h13}" />
         </geometry>
-	<contact_coefficients mu="1" kp="10.0" kd="10.0"/>
+    <contact_coefficients mu="1" kp="10.0" kd="10.0"/>
       </collision>
     </link>
@@ -109,5 +111,5 @@
           <box size="${l} ${e} ${h13}" />
         </geometry>
-	<contact_coefficients mu="1" kp="10.0" kd="10.0"/>
+    <contact_coefficients mu="1" kp="10.0" kd="10.0"/>
       </collision>
     </link>
@@ -350,81 +352,80 @@
       </joint>
 <!-- Sick laser -->
-      <link name="laser_link">
-	<collision>
-	  <origin xyz="0 0 0" rpy="0 0 0"/>
-	  <geometry>
-	    <box size="${x_sick} ${y_sick} ${z_sick}"/>
-	  </geometry>
-	</collision>
-	<visual>
-	  <origin xyz="0 0 0" rpy="0 0 0"/>
-	  <geometry>
+      <link name="safety_laser_base_link">
+    <collision>
+      <origin xyz="0 0 0" rpy="0 0 0"/>
+      <geometry>
+        <box size="${x_sick} ${y_sick} ${z_sick}"/>
+      </geometry>
+    </collision>
+    <visual>
+      <origin xyz="0 0 0" rpy="0 0 0"/>
+      <geometry>
             <mesh filename="package://cititruck_description/meshes/sick_s300_laser.dae"/>
-	  </geometry>
-	</visual>
-	<inertial>
-	  <mass value="1e-5" />
-	  <origin xyz="0 0 0" rpy="0 0 0"/>
-	  <inertia ixx="1e-6" ixy="0" ixz="0" iyy="1e-6" iyz="0" izz="1e-6" />
-	</inertial>
-      </link>
-      <joint name="laser_joint" type="fixed">
-	<axis xyz="0 1 0" />
-	<origin xyz="${l2 + x -y_sick/2.0} 0 ${z_sick/2.0}" rpy="3.14159 0 0"/>
-	<parent link="base_link"/>
-	<child link="laser_link"/>
-      </joint>
+      </geometry>
+    </visual>
+    <inertial>
+      <mass value="1e-5" />
+      <origin xyz="0 0 0" rpy="0 0 0"/>
+      <inertia ixx="1e-6" ixy="0" ixz="0" iyy="1e-6" iyz="0" izz="1e-6" />
+    </inertial>
+      </link>
+      <joint name="safety_laser_joint" type="fixed">
+    <axis xyz="0 1 0" />
+    <origin xyz="${l2 + x -y_sick/2.0} 0 ${z_sick/2.0}" rpy="3.14159 0 0"/>
+    <parent link="base_link"/>
+    <child link="safety_laser_base_link"/>
+      </joint>
+      <sensor_calibration_assembly sensor_id="safety_laser" parent_link="safety_laser_base_link"/>
 <!-- Kinect V2 -->
-    <joint name="kinect_joint" type="fixed">
+    <joint name="kinect2_joint" type="fixed">
       <origin xyz="${-x_pilar/2 + 0.27} ${y_sensor_platform/2.0 - 0.3} ${b1 + 0.6 + z_sensor_bar + 0.05}" rpy="0 0 0" /> <!-- check sensor height z -->
       <parent link="base_pilar"/>
-      <child link="kinect_link"/>
-    </joint>
-    <link name="kinect_link">
-      <visual>
-	<origin xyz="0 0 0" rpy="0 0 ${M_PI}" />
-	<geometry>
-	  <mesh filename="package://cititruck_description/meshes/kinect_v2.dae"/>
-	</geometry>
-      </visual>
-      <collision>
-	<origin xyz="0 0 0" rpy="0 0 0" />
-	<geometry>
-	      <box size="0.1 0.1 0.1"/> <!-- check this later -->
-	</geometry>
-      </collision>
-    </link>
-<!--    <joint name="kinect_depth_joint" type="fixed">
-      <origin xyz="0.0 -0.02 0.0" rpy="0 0 0" />
-      <parent link="kinect_link" />
-      <child link="kinect_depth_frame"/>
-    </joint>
-    <link name="kinect_depth_frame"/>
-    <joint name="kinect_depth_optical_joint" type="fixed">
-      <origin xyz="0 0 0" rpy="${-M_PI/2} 0.0 ${-M_PI/2}" />
-      <parent link="kinect_depth_frame" />
-      <child link="kinect_depth_optical_frame"/>
-    </joint>
-    <link name="kinect_depth_optical_frame"/>
-    <joint name="kinect_rgb_joint" type="fixed">
-      <origin xyz="0.0 -0.0125 0.0" rpy="0 0 0" />
-      <parent link="kinect_link" />
-      <child link="kinect_rgb_frame"/>
-    </joint>
-    <link name="kinect_rgb_frame"/>
-    <joint name="kinect_rgb_optical_joint" type="fixed">
-      <origin xyz="0 0 0" rpy="${-M_PI/2.0} 0.0 ${-M_PI/2.0}" />
-      <parent link="kinect_rgb_frame" />
-      <child link="kinect_rgb_optical_frame"/>
-    </joint>
-    <link name="kinect_rgb_optical_frame"/>-->
+      <child link="kinect2_base_link"/>
+    </joint>
+    <link name="kinect2_base_link"/>
+    <sensor_calibration_assembly sensor_id="kinect2" parent_link="kinect2_base_link" create_final_link="false"/>
+    <link name="kinect2_link">
+      <visual>
+    <origin xyz="0 0 0" rpy="0 0 ${M_PI}" />
+    <geometry>
+      <mesh filename="package://cititruck_description/meshes/kinect_v2.dae"/>
+    </geometry>
+      </visual>
+      <!--
+      <collision>
+    <origin xyz="0 0 0" rpy="0 0 0" />
+    <geometry>
+          <box size="0.1 0.1 0.1"/>
+    </geometry>
+      </collision>-->
+    </link>
 <!-- Velodyne HDL32E -->
-    <!-- FIXME: origin z -->
-    <joint name="velodyne_base_mount_joint" type="fixed">
-      <origin xyz="${-x_pilar/2 + 0.27} ${y_sensor_platform/2.0 - 0.18} ${b1 + 0.6 + z_sensor_bar + 0.14}" rpy="0 0 0"/>
+    <joint name="velodyne_base_joint" type="fixed">
+      <origin xyz="${-x_pilar/2 + 0.27} ${y_sensor_platform/2.0 - 0.18} ${b1 + 0.6 + z_sensor_bar + 0.14 + 0.09081}" rpy="0 0 0"/>
       <parent link="base_pilar"/>
       <child link="velodyne_base_link"/>
     </joint>
-    <link name="velodyne_base_link">
+    <link name="velodyne_base_link"/>
+    <sensor_calibration_assembly sensor_id="velodyne" parent_link="velodyne_base_link" create_final_link="false"/>
+    <link name="velodyne_link">
+      <inertial>
+        <mass value="0.01"/>
+        <origin xyz="0 0 0"/>
+        <inertia ixx="1e-7" ixy="0" ixz="0" iyy="1e-7" iyz="0" izz="1e-7"/>
+      </inertial>
+      <visual>
+        <origin xyz="0 0 -0.09081" rpy="0 0 0" />
+        <geometry>
+          <mesh filename="package://cititruck_description/meshes/HDL32E_scan.dae" />
+        </geometry>
+      </visual>
+    </link>
+    <joint name="velodyne_mount_joint" type="fixed" >
+      <origin xyz="0 0 -0.09081" rpy="0 0 0" />
+      <parent link="velodyne_link" />
+      <child link="velodyne_mount_link"/>
+    </joint>
+    <link name="velodyne_mount_link">
       <inertial>
         <mass value="1.0"/>
@@ -439,4 +440,5 @@
         </geometry>
       </visual>
+      <!--
       <collision>
         <origin rpy="0 0 0" xyz="0 0 0.07212"/>
@@ -445,32 +447,15 @@
         </geometry>
       </collision>
-    </link>
-    <joint name="velodyne_base_scan_joint" type="fixed" >
-      <origin xyz="0 0 0.09081" rpy="0 0 0" />
-      <parent link="velodyne_base_link" />
-      <child link="velodyne"/>
-    </joint>
-    <link name="velodyne">
-      <inertial>
-        <mass value="0.01"/>
-        <origin xyz="0 0 0"/>
-        <inertia ixx="1e-7" ixy="0" ixz="0" iyy="1e-7" iyz="0" izz="1e-7"/>
-      </inertial>
-      <visual>
-        <origin xyz="0 0 -0.09081" rpy="0 0 0" />
-        <geometry>
-          <mesh filename="package://cititruck_description/meshes/HDL32E_scan.dae" />
-        </geometry>
-      </visual>
+  -->
     </link>
     <!-- Asus camera Up -->
-    <!-- FIXME: origin -->
     <joint name="asus_joint" type="fixed">
         <origin xyz="0 ${y_sensor_platform/2.0 + .06} ${b1 + .6 + z_sensor_bar}" rpy="0 0 ${M_PI/2}"/>
         <parent link="base_pilar"/>
-        <child link="asus_link"/>
-      </joint>
-      <link name="asus_link"/>
-      <link name="asus_link_pitch">
+        <child link="asus_base_link"/>
+      </joint>
+      <link name="asus_base_link"/>
+      <sensor_calibration_assembly sensor_id="asus" parent_link="asus_base_link" create_final_link="false"/>
+      <link name="asus_link">
         <inertial>
           <mass value="0.200" />
@@ -484,50 +469,23 @@
           </geometry>
         </visual>
-      <collision>
-	<origin xyz="0 0 0" rpy="0 0 0" />
-	<geometry>
-	  <box size="0.035 0.185 0.025"/>
-	</geometry>
-      </collision>
-      </link>
-      <joint name="asus_joint_pitch" type="revolute">
-        <origin xyz="0 0 0" rpy="0 0 0"/>
-        <parent link="asus_link"/>
-        <child link="asus_link_pitch"/>
-	<axis xyz="0 1 0"/>
-        <limit effort="100" lower="${-M_PI}" upper="${M_PI}" velocity=".1" />
-      </joint>
-<!--      <joint name="asus_depth_joint" type="fixed">
-        <origin xyz="0.0 0.049 0.0" rpy="0 0 0" />
-        <parent link="asus_link" />
-        <child link="asus_depth_frame"/>
-      </joint>
-      <link name="asus_depth_frame"/>
-      <joint name="asus_depth_optical_joint" type="fixed">
-        <origin xyz="0 0 0" rpy="${-M_PI/2} 0.0 ${-M_PI/2}" />
-        <parent link="asus_depth_frame" />
-        <child link="asus_depth_optical_frame"/>
-      </joint>
-      <link name="asus_depth_optical_frame"/>
-      <joint name="asus_rgb_joint" type="fixed">
-        <origin xyz="0.0 0.022 0.0" rpy="0 0 0" />
-        <parent link="asus_link" />
-        <child link="asus_rgb_frame"/>
-      </joint>
-      <link name="asus_rgb_frame"/>
-      <joint name="asus_rgb_optical_joint" type="fixed">
-        <origin xyz="0 0 0" rpy="${-M_PI/2} 0.0 ${-M_PI/2}" />
-        <parent link="asus_rgb_frame" />
-        <child link="asus_rgb_optical_frame"/>
-      </joint>
-  <link name="asus_rgb_optical_frame"/>-->
-  <!-- Asus camera down -->
+            <!--
+          <collision>
+        <origin xyz="0 0 0" rpy="0 0 0" />
+        <geometry>
+          <box size="0.035 0.185 0.025"/>
+        </geometry>
+          </collision>
+        -->
+    </link>
+  <!-- Intel Realsense camera on fork -->
     <!-- FIXME: origin -->
-    <joint name="intel_joint" type="fixed">
+    <joint name="realsense_joint" type="fixed">
         <origin xyz="${l/2} 0 0.235" rpy="0 0 ${M_PI}"/>
         <parent link="base_fork"/>
-        <child link="intel_link"/>
-      </joint>
-      <link name="intel_link">
+        <child link="realsense_base_link"/>
+      </joint>
+      <link name="realsense_base_link"/>
+      <sensor_calibration_assembly sensor_id="realsense" parent_link="realsense_base_link" create_final_link="false"/>
+    <link name="realsense_link">
         <inertial>
           <mass value="0.200" />
@@ -541,35 +499,12 @@
           </geometry>
         </visual>
-      <collision>
-	<origin xyz="0 0 0" rpy="0 0 0" />
-	<geometry>
-	  <box size="0.035 0.185 0.025"/>
-	</geometry>
-      </collision>
-      </link>
-<!--      <joint name="intel_depth_joint" type="fixed">
-        <origin xyz="0.0 0.049 0.0" rpy="0 0 0" />
-        <parent link="intel_link" />
-        <child link="intel_depth_frame"/>
-      </joint>
-      <link name="intel_depth_frame"/>
-      <joint name="intel_depth_optical_joint" type="fixed">
-        <origin xyz="0 0 0" rpy="${-M_PI/2} 0.0 ${-M_PI/2}" />
-        <parent link="intel_depth_frame" />
-        <child link="intel_depth_optical_frame"/>
-      </joint>
-      <link name="intel_depth_optical_frame"/>
-      <joint name="intel_rgb_joint" type="fixed">
-        <origin xyz="0.0 0.022 0.0" rpy="0 0 0" />
-        <parent link="intel_link" />
-        <child link="intel_rgb_frame"/>
-      </joint>
-      <link name="intel_rgb_frame"/>
-      <joint name="intel_rgb_optical_joint" type="fixed">
-        <origin xyz="0 0 0" rpy="${-M_PI/2} 0.0 ${-M_PI/2}" />
-        <parent link="intel_rgb_frame" />
-        <child link="intel_rgb_optical_frame"/>
-      </joint>
-  <link name="intel_rgb_optical_frame"/>-->
+        <!--
+      <collision>
+    <origin xyz="0 0 0" rpy="0 0 0" />
+    <geometry>
+      <box size="0.035 0.185 0.025"/>
+    </geometry>
+      </collision>  -->
+      </link>
     <!-- Reflex camera -->
     <!-- FIXME: origin -->
@@ -577,28 +512,24 @@
         <origin xyz="0 .09 1.90" rpy="0 0 ${M_PI}"/>
         <parent link="base_pilar"/>
-        <child link="reflex_link"/>
-      </joint>
-      <link name="reflex_link"/>
-      <joint name="reflex_joint_pitch" type="revolute">
-        <origin xyz="0 0 0" rpy="0 0 0"/>
-        <parent link="reflex_link"/>
-        <child link="reflex_link_pitch"/>
-	<axis xyz="0 1 0"/>
-        <limit effort="100" lower="${-M_PI}" upper="${M_PI}" velocity=".1" />
-      </joint>
-      <link name="reflex_link_pitch" >
-	<visual>
+        <child link="reflex_base_link"/>
+      </joint>
+      <link name="reflex_base_link"/>
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