Commit message: Extend rotation range of RPY sensor calib joints

File: gazebo_oru/cititruck/cititruck_description/urdf/sensor_calibration_assembly.xacro (robot description, xacro)
@@ -31,5 +31,5 @@
         <!-- Joint limits (only used for version with movable joints) -->
         <xacro:property name="max_trans" value="1.0"/>
-        <xacro:property name="max_rot" value="1.57"/>
+        <xacro:property name="max_rot" value="3.14159"/>
         <!-- Version with fixed pre-calibrated joints (for use in Gazebo and on the actual robot) -->
         <xacro:if value="$(arg use_fixed_joints)">

Commit message: In calibration macro/script, make final sensor link configurable (for Kinect v2)

File: gazebo_oru/cititruck/cititruck_description/urdf/sensor_calibration_assembly.xacro (robot description, xacro)
@@ -47,5 +47,5 @@
     </xacro:macro>
     <!-- Invoke this macro to create a sensor calibration assembly (XYZ offset + rotation + XYZ post-offset). -->
-    <xacro:macro name="sensor_calibration_assembly" params="sensor_id parent_link create_final_link:=true">
+    <xacro:macro name="sensor_calibration_assembly" params="sensor_id parent_link create_final_link:=true final_link_suffix:='link'">
         <!-- Lighter version with a single fixed pre-calibrated joint per sensor (for use in Gazebo and on the actual robot) -->
         <xacro:if value="$(arg use_fixed_joints)">
@@ -59,5 +59,5 @@
                 <origin xyz="${xyz}" rpy="${rpy}"/>
                 <parent link="${parent_link}"/>
-                <child link="${sensor_id}_link"/>
+                <child link="${sensor_id}_${final_link_suffix}"/>
             </joint>
         </xacro:if>
@@ -145,5 +145,5 @@
             <joint name="${sensor_id}_calib_end_link" type="fixed">
                 <parent link="${sensor_id}_calib_post_z_link"/>
-                <child link="${sensor_id}_link"/>
+                <child link="${sensor_id}_${final_link_suffix}"/>
             </joint>
             <!-- End of version with movable joints for calib -->
@@ -151,5 +151,5 @@
         <!-- Final link -->
         <xacro:if value="${create_final_link}">
-            <simple_link name="${sensor_id}_link"/>
+            <simple_link name="${sensor_id}_${final_link_suffix}"/>
         </xacro:if>
     </xacro:macro>
