Commit message: added launchfile for illiad single truck

File: gazebo_oru/cititruck/cititruck_description/urdf/cititruck.xacro (robot description, xacro)
@@ -19,4 +19,8 @@
       <parent link="base_footprint"/>
     </joint>
+    <xacro:include filename="$(find velodyne_description)/urdf/VLP-16.urdf.xacro"/>
+    <VLP-16 parent="base_link" prefix="robot1" name="velodyne" topic="/velodyne_points" hz="10" samples="440">
+      <origin xyz="0.8 0 0.85" rpy="0 0 0" />
+    </VLP-16>
   <!-- Base Link -->
   <link name="base_link">

Commit message: modified cititruck description for kinect camera in simulation, testing pallet detection

File: gazebo_oru/cititruck/cititruck_description/urdf/cititruck.xacro (robot description, xacro)
@@ -304,4 +304,5 @@
       <joint name="kinect_joint" type="fixed">
 	<axis xyz="0 1 0" />
+ 	<!--origin xyz="0.5 0 0.7" rpy="${pi/2 + 0.5} 0 ${-pi/2}" /--> <!-- 0 2.5 0 -->
  	<origin xyz="0.5 0 0.7" rpy="0 2.5 0"/> <!-- 0 2.5 0 -->
 <!--  	<origin xyz="0.5 0 0.7" rpy="0 3.14159 0"/> -->
@@ -309,3 +310,10 @@
 	<child link="kinect_link"/>
       </joint>
+      <link name="kinect_rgb_optical_link"/>
+      <joint name="kinect_optical_joint" type="fixed">
+        <axis xyz="0 1 0" />
+        <origin xyz="0.0 0.0 0.0" rpy="${-pi/2} 0 ${-pi/2}"/>
+        <parent link="kinect_link"/>
+        <child link="kinect_rgb_optical_link"/>
+      </joint>
 </robot>

Commit message: Added gazebo9 mods, should compile and run readme examples

File: gazebo_oru/cititruck/cititruck_description/urdf/cititruck.xacro (robot description, xacro)
@@ -162,5 +162,5 @@
           <origin xyz="0 0 0" rpy="1.57 0 0" />
           <geometry>
-            <cylinder radius="0.08" length=".04" />
+            <cylinder radius="0.08" length="0.04" />
           </geometry>
           <material name="black"/>
@@ -169,5 +169,5 @@
           <origin xyz="0 0 0" rpy="1.57 0 0" />
           <geometry>
-            <cylinder radius="0.08" length=".04" />
+            <cylinder radius="0.08" length="0.04" />
           </geometry>
         </collision>
@@ -220,5 +220,5 @@
           <origin xyz="0 0 0" rpy="1.57 0 0" />
           <geometry>
-            <cylinder radius="0.04" length=".08" />
+            <cylinder radius="0.04" length="0.08" />
           </geometry>
           <material name="gray"/>
@@ -227,5 +227,5 @@
           <origin xyz="0 0 0" rpy="1.57 0 0" />
           <geometry>
-            <cylinder radius="0.04" length=".08" />
+            <cylinder radius="0.04" length="0.08" />
           </geometry>
          <!-- <contact_coefficients mu="100" kp="10.0" kd="0.1"/> -->
@@ -247,5 +247,5 @@
           <origin xyz="0 0 0" rpy="1.57 0 0" />
           <geometry>
-            <cylinder radius="0.04" length=".08" />
+            <cylinder radius="0.04" length="0.08" />
           </geometry>
           <material name="gray"/>
@@ -254,5 +254,5 @@
           <origin xyz="0 0 0" rpy="1.57 0 0" />
           <geometry>
-            <cylinder radius="0.04" length=".08" />
+            <cylinder radius="0.04" length="0.08" />
           </geometry>
          <!-- <contact_coefficients mu="100" kp="10.0" kd="0.1"/> -->

File: gazebo_oru/cititruck/cititruck_description/urdf/cititruck_air.xacro (robot description, xacro)
@@ -210,5 +210,5 @@
           <origin xyz="0 0 0" rpy="1.57 0 0" />
           <geometry>
-            <cylinder radius="0.04" length=".08" />
+            <cylinder radius="0.04" length="0.08" />
           </geometry>
           <material name="gray"/>
@@ -217,5 +217,5 @@
           <origin xyz="0 0 0" rpy="1.57 0 0" />
           <geometry>
-            <cylinder radius="0.04" length=".08" />
+            <cylinder radius="0.04" length="0.08" />
           </geometry>
          <!-- <contact_coefficients mu="100" kp="10.0" kd="0.1"/> -->
@@ -237,5 +237,5 @@
           <origin xyz="0 0 0" rpy="1.57 0 0" />
           <geometry>
-            <cylinder radius="0.04" length=".08" />
+            <cylinder radius="0.04" length="0.08" />
           </geometry>
           <material name="gray"/>
@@ -244,5 +244,5 @@
           <origin xyz="0 0 0" rpy="1.57 0 0" />
           <geometry>
-            <cylinder radius="0.04" length=".08" />
+            <cylinder radius="0.04" length="0.08" />
           </geometry>
          <!-- <contact_coefficients mu="100" kp="10.0" kd="0.1"/> -->

File: gazebo_oru/cititruck/cititruck_description/urdf/iliad_velodyne_cititruck.xacro (robot description, xacro)
@@ -243,5 +243,5 @@
             <origin xyz="0 0 0" rpy="1.57 0 0"/>
             <geometry>
-                <cylinder radius="0.04" length=".08"/>
+                <cylinder radius="0.04" length="0.08"/>
             </geometry>
             <material name="gray"/>
@@ -250,5 +250,5 @@
             <origin xyz="0 0 0" rpy="1.57 0 0"/>
             <geometry>
-                <cylinder radius="0.04" length=".08"/>
+                <cylinder radius="0.04" length="0.08"/>
             </geometry>
             <!-- <contact_coefficients mu="100" kp="10.0" kd="0.1"/>-->
@@ -270,5 +270,5 @@
             <origin xyz="0 0 0" rpy="1.57 0 0"/>
             <geometry>
-                <cylinder radius="0.04" length=".08"/>
+                <cylinder radius="0.04" length="0.08"/>
             </geometry>
             <material name="gray"/>
@@ -277,5 +277,5 @@
             <origin xyz="0 0 0" rpy="1.57 0 0"/>
             <geometry>
-                <cylinder radius="0.04" length=".08"/>
+                <cylinder radius="0.04" length="0.08"/>
             </geometry>
             <!-- <contact_coefficients mu="100" kp="10.0" kd="0.1"/>-->
