Commit message: Adding sensor calibration joints for Cititruck. Some cleanup.

File: gazebo_oru/cititruck/cititruck_description/urdf/iliad_velodyne_cititruck.xacro (robot description, xacro)
@@ -4,5 +4,5 @@
     <xacro:arg name="velodyne" default="false"/>
     <xacro:arg name="kinect2" default="false"/>
-    <xacro:arg name="kinect1" default="false"/> <!-- deprecated -->
+    <xacro:arg name="asus" default="false"/> <!-- not used by Cititruck? -->
     <!-- Arguments used in cititruck.gazebo -->
     <xacro:arg name="controller_prefix" default=""/>
@@ -10,9 +10,12 @@
     <xacro:arg name="sick_name" default="safety"/>
     <xacro:arg name="ls2000_name" default="nav"/>
-    <xacro:arg name="kinect2_name" default=""/>
+    <xacro:arg name="kinect2_name" default="kinect2"/>
+    <xacro:arg name="asus_name" default="asus"/>
     <!-- Import all Gazebo-customization elements, including Gazebo colors -->
     <xacro:include filename="$(find cititruck_description)/urdf/cititruck.gazebo"/>
     <!-- Import Rviz colors -->
     <xacro:include filename="$(find cititruck_description)/urdf/materials.xacro"/>
+    <!-- Adds extra joints for calibration of sensors -->
+    <xacro:include filename="$(find cititruck_description)/urdf/sensor_calibration_assembly.xacro" />
     <xacro:property name="forks_pidP" value="2000"/>
     <xacro:property name="forks_pidI" value="0"/>
@@ -287,5 +290,5 @@
     <!-- SENSORS START HERE -->
     <!-- SICK laser -->
-    <link name="$(arg sick_name)_link">
+    <link name="$(arg sick_name)_base_link">
         <collision>
             <origin xyz="0 0 0" rpy="0 0 0"/>
@@ -310,8 +313,9 @@
         <origin xyz="1.4 0 0.02" rpy="3.14159 0 0"/>
         <parent link="base_link"/>
-        <child link="$(arg sick_name)_link"/>
-    </joint>
+        <child link="$(arg sick_name)_base_link"/>
+    </joint>
+    <sensor_calibration_assembly sensor_id="$(arg sick_name)" parent_link="$(arg sick_name)_base_link"/>
     <!-- LS2000 navigation/localization laser -->
-    <link name="$(arg ls2000_name)_link">
+    <link name="$(arg ls2000_name)_base_link">
         <collision>
             <origin xyz="0 0 0" rpy="0 0 0"/>
@@ -335,21 +339,26 @@
         <origin xyz="0.8 0 0.85" rpy="0 0 0"/>
         <parent link="base_link"/>
-        <child link="$(arg ls2000_name)_link"/>
-    </joint>
+        <child link="$(arg ls2000_name)_base_link"/>
+    </joint>
+    <sensor_calibration_assembly sensor_id="$(arg ls2000_name)" parent_link="$(arg ls2000_name)_base_link"/>
     <!-- Velodyne VLP16 -->
+    <!-- FIXME: We should rather attach the calibration assembly to the final link, otherwise we have a 3.7cm z offset during rotation, so need to split up the imported xacro -->
+    <!-- FIXED: The name should be velodyne_link -->
     <xacro:if value="$(arg velodyne)">
       <xacro:include filename="$(find velodyne_description)/urdf/VLP-16.urdf.xacro"/>
-      <VLP-16 parent="base_link" prefix="$(arg tf_prefix)/velodyne" name="velodyne" topic="/velodyne_points" hz="10" samples="440">
-          <origin xyz="0.8 0 0.95" rpy="0 0 0" />
+      <VLP-16 parent="velodyne_base_link" prefix="$(arg tf_prefix)/velodyne" name="velodyne_link" topic="/velodyne_points" hz="10" samples="440">
+          <origin xyz="0 0 0" rpy="0 0 0" /> <!-- given by calibration -->
       </VLP-16>
+      <sensor_calibration_assembly sensor_id="velodyne" parent_link="base_link" final_link_suffix="base_link"/>
     </xacro:if>
     <!-- Kinect v2 -->
     <xacro:if value="$(arg kinect2)">
       <xacro:include filename="$(find kinect2_description)/urdf/kinect2/kinect2.xacro"/>
-      <kinect2_sensor parent="base_link" prefix="$(arg tf_prefix)" name="kinect2" cam_px="0.65" cam_py="0" cam_pz="1.15" cam_or="0" cam_op="0" cam_oy="3.1415926"/>
+      <kinect2_sensor parent="kinect2_base_link" prefix="$(arg tf_prefix)" name="kinect2" cam_px="0" cam_py="0" cam_pz="0" cam_or="0" cam_op="0" cam_oy="3.1415926"/>
+      <sensor_calibration_assembly sensor_id="kinect2" parent_link="base_link" final_link_suffix="base_link"/>
     </xacro:if>
-    <!-- Old Kinect (deprecated, only used for pallet detection?) -->
-    <xacro:if value="$(arg kinect1)">
-      <link name="kinect_link">
+    <!-- Asus for pallet detection (deprecated?) -->
+    <xacro:if value="$(arg asus)">
+      <link name="$(arg asus_name)_base_link">
           <collision>
               <origin xyz="0 0 0" rpy="0 0 0"/>
@@ -370,11 +379,12 @@
           </inertial>
       </link>
-      <joint name="kinect_joint" type="fixed">
+      <joint name="$(arg asus_name)_joint" type="fixed">
           <axis xyz="0 1 0"/>
           <origin xyz="0.5 0 0.7" rpy="0 2.5 0"/> <!-- 0 2.5 0 -->
           <!--        <origin xyz="0.5 0 0.7" rpy="0 3.14159 0"/>-->
           <parent link="base_link"/>
-          <child link="kinect_link"/>
+          <child link="$(arg asus_name)_base_link"/>
       </joint>
+      <sensor_calibration_assembly sensor_id="$(arg asus_name)" parent_link="$(arg asus_name)_base_link"/>
     </xacro:if>
 </robot>

Commit message: Added changes from iliad_uol_cititruck.xacro

File: gazebo_oru/cititruck/cititruck_description/urdf/iliad_velodyne_cititruck.xacro (robot description, xacro)
@@ -10,6 +10,7 @@
     <xacro:arg name="sick_name" default="safety"/>
     <xacro:arg name="ls2000_name" default="nav"/>
-    <xacro:arg name="kinect2_name" default=""/>
-    <xacro:arg name="kinect1_name" default="kinect"/>
+    <xacro:arg name="kinect2_name" default="kinect2"/>
+    <xacro:arg name="asus_name" default="asus"/>
+    <xacro:arg name="is_uol_variant" default="true"/>
     <!-- Import all Gazebo-customization elements, including Gazebo colors -->
     <xacro:include filename="$(find cititruck_description)/urdf/cititruck.gazebo"/>
@@ -24,4 +25,5 @@
     <xacro:property name="forks_high" value="0.2"/>
     <xacro:property name="forks_maxeffort" value="1000"/>
+    <xacro:property name="PI" value="3.141592"/>
     <!-- base_footprint is a fictitious link(frame) that is on the ground right below base_link origin, navigation stack dedpends on this frame and KDL needs a root link without any intertia -->
     <link name="base_footprint"/>
@@ -51,5 +53,6 @@
             <material name="red"/>
         </visual>
-        <!-- Top shelf -->
+	<!-- Top shelf ORU version -->
+    <xacro:unless value="$(arg is_uol_variant)">
         <visual>
             <origin xyz="0.8 0 1.1" rpy="0 0 0" />
@@ -73,4 +76,30 @@
             <material name="red"/>
         </visual>
+    </xacro:unless>
+    <!-- Top Bar UoL version -->
+    <xacro:if value="$(arg is_uol_variant)">
+        <visual>
+            <origin xyz="0.8 0 0.935" rpy="0 0 0" />
+            <geometry>
+                <!-- box size="0.4 0.55 0.03" / -->
+                <box size="0.05 0.54 0.025" />
+            </geometry>
+            <material name="gray"/>
+        </visual>
+        <visual>
+            <origin xyz="0.8 0.26 0.85" rpy="0 0 0" />
+            <geometry>
+                <box size="0.05 0.025 0.18" />
+            </geometry>
+            <material name="gray"/>
+        </visual>
+        <visual>
+            <origin xyz="0.8 -0.26 0.85" rpy="0 0 0" />
+            <geometry>
+                <box size="0.05 0.025 0.18" />
+            </geometry>
+            <material name="gray"/>
+        </visual>
+    </xacro:if>
     </link>
     <!-- Forks -->
@@ -147,5 +176,6 @@
         <child link="base_fork"/>
         <axis xyz="0 0 1"/>
-        <limit effort="1000" lower="-1" upper="1" velocity="100"/>
+        <!-- lower was -1, making it collide with the wheels-->
+        <limit effort="1000" lower="0.05" upper="1" velocity="100"/>
     </joint>
     <!-- Steering -->
@@ -243,12 +273,12 @@
             <origin xyz="0 0 0" rpy="1.57 0 0"/>
             <geometry>
-                <cylinder radius="0.04" length="0.08"/>
-            </geometry>
-            <material name="gray"/>
-        </visual>
-        <collision>
-            <origin xyz="0 0 0" rpy="1.57 0 0"/>
-            <geometry>
-                <cylinder radius="0.04" length="0.08"/>
+                <cylinder radius="0.04" length=".08"/>
+            </geometry>
+            <material name="gray"/>
+        </visual>
+        <collision>
+            <origin xyz="0 0 0" rpy="1.57 0 0"/>
+            <geometry>
+                <cylinder radius="0.04" length=".08"/>
             </geometry>
             <!-- <contact_coefficients mu="100" kp="10.0" kd="0.1"/>-->
@@ -270,12 +300,12 @@
             <origin xyz="0 0 0" rpy="1.57 0 0"/>
             <geometry>
-                <cylinder radius="0.04" length="0.08"/>
-            </geometry>
-            <material name="gray"/>
-        </visual>
-        <collision>
-            <origin xyz="0 0 0" rpy="1.57 0 0"/>
-            <geometry>
-                <cylinder radius="0.04" length="0.08"/>
+                <cylinder radius="0.04" length=".08"/>
+            </geometry>
+            <material name="gray"/>
+        </visual>
+        <collision>
+            <origin xyz="0 0 0" rpy="1.57 0 0"/>
+            <geometry>
+                <cylinder radius="0.04" length=".08"/>
             </geometry>
             <!-- <contact_coefficients mu="100" kp="10.0" kd="0.1"/>-->
@@ -347,18 +377,20 @@
     <xacro:if value="$(arg velodyne)">
       <xacro:include filename="$(find velodyne_description8)/urdf/VLP-16.urdf.xacro"/>
-      <VLP-16 parent="base_link" gpu="true" name="velodyne" topic="/$(arg tf_prefix)/$(arg sensor_prefix)/velodyne/velodyne_points" hz="10" samples="440">
-          <origin xyz="0.8 0 0.95" rpy="0 0 0" />
+      <VLP-16 parent="velodyne_base_link" gpu="true" name="velodyne" topic="/$(arg tf_prefix)/$(arg sensor_prefix)/velodyne/velodyne_points" hz="10" samples="440">
+          <origin xyz="0 0 0" rpy="0 0 0" />
       </VLP-16>
-      <sensor_calibration_assembly sensor_id="velodyne" parent_link="base_link" final_link_suffix="base_link"/>
+     <sensor_calibration_assembly sensor_id="velodyne" parent_link="base_link" final_link_suffix="base_link"/>
     </xacro:if>
     <!-- Kinect v2 -->
     <xacro:if value="$(arg kinect2)">
-      <xacro:include filename="$(find kinect2_description)/urdf/kinect2/kinect2.xacro"/>
-      <kinect2_sensor parent="base_link" prefix="/$(arg tf_prefix)/$(arg sensor_prefix)" name="kinect2" cam_px="0.65" cam_py="0" cam_pz="1.15" cam_or="0" cam_op="0" cam_oy="3.1415926"/>
+    <xacro:include filename="$(find kinect2_description)/urdf/kinect2/kinect2.xacro"/>
+      <kinect2_sensor parent="kinect2_base_link" prefix="$(arg tf_prefix)/$(arg sensor_prefix)" name="kinect2" cam_px="0" cam_py="0" cam_pz="0" cam_or="0" cam_op="0" cam_oy="0"/>
+      <sensor_calibration_assembly sensor_id="kinect2" parent_link="base_link" final_link_suffix="base_link"/>
     </xacro:if>
-    <!-- Old Kinect, only used for pallet detection -->
-    <xacro:if value="$(arg kinect1)">
+    <!-- Asus for pallet detection -->
+    <xacro:if value="$(arg asus)">
       <xacro:include filename="$(find asus_description)/urdf/asus/asus.xacro"/>
-      <asus_sensor parent="base_link" prefix="/$(arg tf_prefix)/$(arg sensor_prefix)" name="$(arg kinect1_name)" cam_px="0.55" cam_py="0" cam_pz="0.7" cam_or="0" cam_op="2.5" cam_oy="0"/>
+      <asus_sensor parent="$(arg asus_name)_base_link" prefix="$(arg tf_prefix)/$(arg sensor_prefix)"  name="$(arg asus_name)"  cam_px="0" cam_py="0" cam_pz="0" cam_or="0" cam_op="0" cam_oy="0"/>
+      <sensor_calibration_assembly sensor_id="$(arg asus_name)" parent_link="base_link" final_link_suffix="base_link"/>
     </xacro:if>
 </robot>
