Commit message: Apply new naming scheme to sensors of bt_truck

File: gazebo_oru/cititruck/cititruck_description/urdf/bt_truck.xacro (robot description, xacro)
@@ -354,5 +354,5 @@
       </joint>
 <!-- Sick laser -->
-      <link name="safety_laser_base_link">
+      <link name="laser2d_floor_base_link">
     <collision>
       <origin xyz="0 0 0" rpy="0 0 0"/>
@@ -373,11 +373,11 @@
     </inertial>
       </link>
-      <joint name="safety_laser_joint" type="fixed">
+      <joint name="laser2d_floor_joint" type="fixed">
     <axis xyz="0 1 0" />
     <origin xyz="${l2 + x -y_sick/2.0} 0 ${z_sick/2.0}" rpy="3.14159 0 0"/>
     <parent link="base_link"/>
-    <child link="safety_laser_base_link"/>
-      </joint>
-      <sensor_calibration_assembly sensor_id="safety_laser" parent_link="safety_laser_base_link"/>
+    <child link="laser2d_floor_base_link"/>
+      </joint>
+      <sensor_calibration_assembly sensor_id="laser2d_floor" parent_link="laser2d_floor_base_link"/>
 <!-- Kinect V2 -->
     <joint name="kinect2_joint" type="fixed">
@@ -403,5 +403,5 @@
       </collision>-->
     </link>
-<!-- Velodyne HDL32E -->
+<!-- velodyne HDL32E -->
     <joint name="velodyne_base_joint" type="fixed">
       <origin xyz="${-x_pilar/2 + 0.27} ${y_sensor_platform/2.0 - 0.18} ${b1 + 0.6 + z_sensor_bar + 0.14 + 0.09081}" rpy="0 0 0"/>
@@ -452,12 +452,12 @@
     </link>
     <!-- Asus camera Up -->
-    <joint name="asus_joint" type="fixed">
+    <joint name="asus_side_joint" type="fixed">
         <origin xyz="0 ${y_sensor_platform/2.0 + .06} ${b1 + .6 + z_sensor_bar}" rpy="0 0 ${M_PI/2}"/>
         <parent link="base_pilar"/>
-        <child link="asus_base_link"/>
-      </joint>
-      <link name="asus_base_link"/>
-      <sensor_calibration_assembly sensor_id="asus" parent_link="asus_base_link" create_final_link="false"/>
-      <link name="asus_link">
+        <child link="asus_side_base_link"/>
+      </joint>
+      <link name="asus_side_base_link"/>
+      <sensor_calibration_assembly sensor_id="asus_side" parent_link="asus_side_base_link" create_final_link="false"/>
+      <link name="asus_side_link">
         <inertial>
           <mass value="0.200" />
@@ -482,12 +482,12 @@
   <!-- Intel Realsense camera on fork -->
     <!-- FIXME: origin -->
-    <joint name="realsense_joint" type="fixed">
+    <joint name="realsense_fork_joint" type="fixed">
         <origin xyz="${l/2} 0 0.235" rpy="0 0 ${M_PI}"/>
         <parent link="base_fork"/>
-        <child link="realsense_base_link"/>
-      </joint>
-      <link name="realsense_base_link"/>
-      <sensor_calibration_assembly sensor_id="realsense" parent_link="realsense_base_link" create_final_link="false"/>
-    <link name="realsense_link">
+        <child link="realsense_fork_base_link"/>
+      </joint>
+      <link name="realsense_fork_base_link"/>
+      <sensor_calibration_assembly sensor_id="realsense_fork" parent_link="realsense_fork_base_link" create_final_link="false"/>
+    <link name="realsense_fork_link">
         <inertial>
           <mass value="0.200" />

Commit message: Pushing results from integration week: Fixing calibration when using fixed joints; adding save_calibration script; renaming LS2000->laser_top; adding calibration joint for laser2d_top; first very rough calibration of Velodyne and 2D lasers on bt_truck.

File: gazebo_oru/cititruck/cititruck_description/urdf/bt_truck.xacro (robot description, xacro)
@@ -391,5 +391,5 @@
       </link>
 <!-- LS2000 -->
-      <link name="LS2000_link">
+      <link name="laser2d_top_base_link">
         <inertial>
           <mass value="0.200" />
@@ -412,8 +412,9 @@
         -->
     </link>
-      <joint name="LS2000_joint" type="fixed">
+      <joint name="laser2d_top_base_joint" type="fixed">
         <origin xyz="1.257 0 2.3005" rpy="0 0 ${M_PI}"/>
         <parent link="base_link"/>
-        <child link="LS2000_link"/>
-      </joint>
+        <child link="laser2d_top_base_link"/>
+      </joint>
+      <sensor_calibration_assembly sensor_id="laser2d_top" parent_link="laser2d_top_base_link"/>
 </robot>

File: gazebo_oru/cititruck/cititruck_description/urdf/sensor_calibration_assembly.xacro (robot description, xacro)
@@ -1,3 +1,23 @@
 <?xml version="1.0"?>
+<!--
+# (c) 2018 EU H2020 Project ILIAD, iliad-project.eu
+# The following code in this file is licensed under the MIT license:
+#
+# Permission is hereby granted, free of charge, to any person obtaining a copy
+# of this software and associated documentation files (the "Software"), to deal
+# in the Software without restriction, including without limitation the rights
+# to use, copy, modify, merge, publish, distribute, sublicense, and/or sell
+# copies of the Software, and to permit persons to whom the Software is
+# furnished to do so, subject to the following conditions:
+# The above copyright notice and this permission notice shall be included in all
+# copies or substantial portions of the Software.
+# THE SOFTWARE IS PROVIDED "AS IS", WITHOUT WARRANTY OF ANY KIND, EXPRESS OR
+# IMPLIED, INCLUDING BUT NOT LIMITED TO THE WARRANTIES OF MERCHANTABILITY,
+# FITNESS FOR A PARTICULAR PURPOSE AND NONINFRINGEMENT. IN NO EVENT SHALL THE
+# AUTHORS OR COPYRIGHT HOLDERS BE LIABLE FOR ANY CLAIM, DAMAGES OR OTHER
+# LIABILITY, WHETHER IN AN ACTION OF CONTRACT, TORT OR OTHERWISE, ARISING FROM,
+# OUT OF OR IN CONNECTION WITH THE SOFTWARE OR THE USE OR OTHER DEALINGS IN THE
+# SOFTWARE.
+-->
 <!-- This xacro contains a macro for spawning a sensor calibration assembly inside a robot's URDF file.
  The idea is that on the final robot, the assembly just consists of two fixed joints, which have the origin and rpy values set properly
@@ -5,6 +25,5 @@
  Instead, during the calibration phase, these two fixed joints are replaced by a chain of nine prismatic+revolute joints, such that
  each dimension can be tweaked individually using the sliders in the joint state publisher GUI.
- Once calibrated, the slider positions should be (manually) copied into a text file, to be read either by the joint state publisher
- during subsequent runs (as zero positions of the joints), or to be used as calibration values for the fixed joints in this macro.
+ Once calibrated, calibration values should be saved via save_calibration.py.
 -->
 <robot name="sensor_calibration_assembly_macro" xmlns:xacro="http://ros.org/wiki/xacro">
@@ -29,31 +48,15 @@
     <!-- Invoke this macro to create a sensor calibration assembly (XYZ offset + rotation + XYZ post-offset). -->
     <xacro:macro name="sensor_calibration_assembly" params="sensor_id parent_link create_final_link:=true">
-        <!-- Joint limits (only used for version with movable joints) -->
-        <xacro:property name="max_trans" value="1.0"/>
-        <xacro:property name="max_rot" value="3.14159"/>
-        <!-- Version with fixed pre-calibrated joints (for use in Gazebo and on the actual robot) -->
+        <!-- Lighter version with a single fixed pre-calibrated joint per sensor (for use in Gazebo and on the actual robot) -->
         <xacro:if value="$(arg use_fixed_joints)">
-            <!-- Load joint zero positions, and use them for the fixed offsets and rpy -->
-            <xacro:property name="default_calib" value="${load_yaml('$(arg calib_file)')['zeros']}"/>
-            <xacro:property name="pre_x" value="${default_calib.get(sensor_id + '_calib_pre_x', 0.0)}"/>
-            <xacro:property name="pre_y" value="${default_calib.get(sensor_id + '_calib_pre_y', 0.0)}"/>
-            <xacro:property name="pre_z" value="${default_calib.get(sensor_id + '_calib_pre_z', 0.0)}"/>
-            <xacro:property name="roll"  value="${default_calib.get(sensor_id + '_calib_roll', 0.0)}"/>
-            <xacro:property name="pitch" value="${default_calib.get(sensor_id + '_calib_pitch', 0.0)}"/>
-            <xacro:property name="yaw"   value="${default_calib.get(sensor_id + '_calib_yaw', 0.0)}"/>
-            <xacro:property name="post_x" value="${default_calib.get(sensor_id + '_calib_post_x', 0.0)}"/>
-            <xacro:property name="post_y" value="${default_calib.get(sensor_id + '_calib_post_y', 0.0)}"/>
-            <xacro:property name="post_z" value="${default_calib.get(sensor_id + '_calib_post_z', 0.0)}"/>
-            <!-- Initial offset (pre-translation) + Rotation -->
-            <simple_link name="${sensor_id}_calib_link"/>
-            <joint name="${parent_link}_to_${sensor_id}_calib_link" type="fixed">
-                <origin xyz="${pre_x} ${pre_y} ${pre_z}" rpy="${roll} ${pitch} ${yaw}"/>
+            <!-- Load resulting transforms exported by save_calibration.py, and use them for the fixed offset and rpy -->
+            <xacro:property name="all_sensor_tfs" value="${load_yaml('$(arg calib_file)').get('resulting_transforms', dict())}"/>
+            <xacro:property name="sensor_tf" value="${all_sensor_tfs.get(sensor_id, [0.0]*6)}"/>
+            <xacro:property name="xyz" value="${' '.join(str(x) for x in sensor_tf[0:3] )}"/>
+            <xacro:property name="rpy" value="${' '.join(str(x) for x in sensor_tf[3:6] )}"/>
+            <!-- Resulting transform -->
+            <joint name="${sensor_id}_resulting_transform_joint" type="fixed">
+                <origin xyz="${xyz}" rpy="${rpy}"/>
                 <parent link="${parent_link}"/>
-                <child link="${sensor_id}_calib_link"/>
-            </joint>
-            <!-- Final offset (post-translation after rotation) -->
-            <joint name="${sensor_id}_calib_link_to_${sensor_id}_link" type="fixed">
-                <origin xyz="${post_x} ${post_y} ${post_z}"/>
-                <parent link="${sensor_id}_calib_link"/>
                 <child link="${sensor_id}_link"/>
             </joint>
@@ -61,5 +64,15 @@
         <!-- Version with movable joints (only for calib use with joint state publisher GUI) -->
         <xacro:unless value="$(arg use_fixed_joints)">
+            <!-- Dynamic joint limits -->
+            <xacro:property name="max_trans" value="1.0"/>
+            <xacro:property name="max_rot" value="3.14159"/>
             <!-- Zero values will be loaded by joint state publisher! Joints should be 1D because only 1D values are supported in the GUI -->
+            <!-- Initial dummy link (zero transform) that starts the chain -->
+            <!-- Do not remove, required for automatic saving! -->
+            <simple_link name="${sensor_id}_calib_start_link"/>
+            <joint name="${sensor_id}_calib_start" type="fixed">
+                <parent link="${parent_link}"/>
+                <child link="${sensor_id}_calib_start_link"/>
+            </joint>
             <!-- Pre-translation -->
             <simple_link name="${sensor_id}_calib_pre_x_link"/>
@@ -67,5 +80,5 @@
                 <axis xyz="1 0 0"/>
                 <limit lower="-${max_trans}" upper="+${max_trans}" effort="1" velocity="1"/>
-                <parent link="${parent_link}"/>
+                <parent link="${sensor_id}_calib_start_link"/>
                 <child link="${sensor_id}_calib_pre_x_link"/>
             </joint>
@@ -99,10 +112,10 @@
                 <child link="${sensor_id}_calib_pitch_link"/>
             </joint>
-            <simple_link name="${sensor_id}_calib_link"/>
+            <simple_link name="${sensor_id}_calib_yaw_link"/>
             <joint name="${sensor_id}_calib_yaw" type="revolute">
                 <axis xyz="0 0 1"/>
                 <limit lower="-${max_rot}" upper="+${max_rot}" effort="1" velocity="1"/>
                 <parent link="${sensor_id}_calib_pitch_link"/>
-                <child link="${sensor_id}_calib_link"/>
+                <child link="${sensor_id}_calib_yaw_link"/>
             </joint>
             <!-- Post-translation (after rotation) -->
@@ -111,5 +124,5 @@
                 <axis xyz="1 0 0"/>
                 <limit lower="-${max_trans}" upper="+${max_trans}" effort="1" velocity="1"/>
-                <parent link="${sensor_id}_calib_link"/>
+                <parent link="${sensor_id}_calib_yaw_link"/>
                 <child link="${sensor_id}_calib_post_x_link"/>
             </joint>
@@ -121,12 +134,20 @@
                 <child link="${sensor_id}_calib_post_y_link"/>
             </joint>
+            <simple_link name="${sensor_id}_calib_post_z_link"/>
             <joint name="${sensor_id}_calib_post_z" type="prismatic">
                 <axis xyz="0 0 1"/>
                 <limit lower="-${max_trans}" upper="+${max_trans}" effort="1" velocity="1"/>
                 <parent link="${sensor_id}_calib_post_y_link"/>
+                <child link="${sensor_id}_calib_post_z_link"/>
+            </joint>
+            <!-- Final dummy link (zero transform) that ends the chain -->
+            <!-- Do not remove, required for automatic saving! -->
+            <joint name="${sensor_id}_calib_end_link" type="fixed">
+                <parent link="${sensor_id}_calib_post_z_link"/>
                 <child link="${sensor_id}_link"/>
             </joint>
             <!-- End of version with movable joints for calib -->
         </xacro:unless>
+        <!-- Final link -->
         <xacro:if value="${create_final_link}">
             <simple_link name="${sensor_id}_link"/>

Commit message: Rough Kinect v2 calibration on bt_truck, had to add one extra joint, needs to be verified on real hardware

File: gazebo_oru/cititruck/cititruck_description/urdf/bt_truck.xacro (robot description, xacro)
@@ -237,25 +237,25 @@
 <!-- Kinect V2 -->
     <joint name="kinect2_joint" type="fixed">
-      <origin xyz="${ 0.27 + x } ${y_sensor_platform/2.0 - 0.3} ${b1 + 0.6 + z_sensor_bar + 0.05}" rpy="0 0 0" /> <!-- check sensor height z -->
+      <origin xyz="${ 0.27 + x } ${y_sensor_platform/2.0 - 0.3} ${b1 + 0.6 + z_sensor_bar + 0.05}" rpy="0 0 ${M_PI}" /> <!-- check sensor height z -->
       <parent link="base_link"/>
       <child link="kinect2_base_link"/>
     </joint>
-    <link name="kinect2_base_link"/>
-    <sensor_calibration_assembly sensor_id="kinect2" parent_link="kinect2_base_link" create_final_link="false"/>
-    <link name="kinect2_link">
-      <visual>
-    <origin xyz="0 0 0" rpy="0 0 ${M_PI}" />
-    <geometry>
-      <mesh filename="package://cititruck_description/meshes/kinect_v2.dae"/>
-    </geometry>
-      </visual>
-      <!--
-      <collision>
-    <origin xyz="0 0 0" rpy="0 0 0" />
-    <geometry>
-          <box size="0.1 0.1 0.1"/>
-    </geometry>
-      </collision>-->
-    </link>
+    <link name="kinect2_base_link">
+        <visual>
+          <origin xyz="0 0 0" rpy="0 0 0" />
+          <geometry>
+            <mesh filename="package://cititruck_description/meshes/kinect_v2.dae"/>
+          </geometry>
+          </visual>
+    </link>
+    <sensor_calibration_assembly sensor_id="kinect2" parent_link="kinect2_base_link" final_link_suffix="before_optical_link"/>
+    <!-- Extra joint added to get pointcloud aligned correctly in bagfiles; do not remove without cross-checking against recorded bagfiles -->
+    <!-- TODO: Check against live data on robot when running kinect2_bridge -->
+    <joint name="kinect2_optical_joint" type="fixed">
+      <origin rpy="${-M_PI/2.0} 0 ${-M_PI/2.0}"/>
+      <parent link="kinect2_before_optical_link"/>
+      <child link="kinect2_link"/>
+    </joint>
+    <link name="kinect2_link"/>
 <!-- Velodyne HDL32E -->
     <joint name="velodyne_base_joint" type="fixed">

Commit message: Update kinect position according to reality

File: gazebo_oru/cititruck/cititruck_description/urdf/bt_truck.xacro (robot description, xacro)
@@ -237,5 +237,5 @@
 <!-- Kinect V2 -->
     <joint name="kinect2_joint" type="fixed">
-      <origin xyz="${ 0.27 + x } ${y_sensor_platform/2.0 - 0.3} ${b1 + 0.6 + z_sensor_bar + 0.05}" rpy="0 0 ${M_PI}" /> <!-- check sensor height z -->
+      <origin xyz="${ 0.3 + x } ${0.29 - y_sensor_platform/2.0} ${b1 + 0.76 + z_sensor_bar + 0.05}" rpy="0 0 ${M_PI}" /> <!-- check sensor height z -->
       <parent link="base_link"/>
       <child link="kinect2_base_link"/>

Commit message: update xacro with extrinsic calibraiton of velodyne, removed connection to manual calibration through gui

File: gazebo_oru/cititruck/cititruck_description/urdf/bt_truck.xacro (robot description, xacro)
@@ -260,10 +260,10 @@
 <!-- Velodyne HDL32E -->
     <joint name="velodyne_base_joint" type="fixed">
-      <origin xyz="${ x + 0.27} ${y_sensor_platform/2.0 - 0.18} ${b1 + 0.6 + z_sensor_bar + 0.14 + 0.09081}" rpy="0 0 0"/>
+      <origin xyz="1.1187 0.1354 ${b1 + 0.6 + z_sensor_bar + 0.14 + 0.09081}" rpy="0 0 1.594682"/>
       <parent link="base_link"/>
-      <child link="velodyne_base_link"/>
-    </joint>
-    <link name="velodyne_base_link"/>
-    <sensor_calibration_assembly sensor_id="velodyne" parent_link="velodyne_base_link" create_final_link="false"/>
+      <child link="velodyne_link"/>
+    </joint>
+    <!--link name="velodyne_base_link"/-- ><!-- removed as extrinsic calibration now exists -->
+    <!--sensor_calibration_assembly sensor_id="velodyne" parent_link="velodyne_base_link" create_final_link="false"/-->
     <link name="velodyne_link">
       <inertial>

Commit message: Manually tuned Velodyne calibration for bt_truck (based upon Daniel's values, where yaw and z were a bit off)

File: gazebo_oru/cititruck/cititruck_description/urdf/bt_truck.xacro (robot description, xacro)
@@ -260,5 +260,5 @@
 <!-- Velodyne HDL32E -->
     <joint name="velodyne_base_joint" type="fixed">
-      <origin xyz="1.1187 0.1354 ${b1 + 0.6 + z_sensor_bar + 0.14 + 0.09081}" rpy="0 0 1.594682"/>
+      <origin xyz="1.10127 -0.1121022 1.75" rpy="0.00234404 -0.00292631 1.49467"/>
       <parent link="base_link"/>
       <child link="velodyne_link"/>
